File: daq_interface.kicad_sch (KiCad schematic)
At the start: 0 parts

Commit message: complete daq interface with digital buffering and analog filtering
Parts:
- added C11, C12, C13: 10nF, symbol Device:C
- added J5: DAQ_IO, symbol Connector_Generic:Conn_01x08
- added R1, R2, R3: 330R, symbol Device:R
- added R4: 100R, symbol Device:R
- added R5, R6: 1k, symbol Device:R
- added TP1, TP2, TP3, TP4, TP5, TP6, TP7, TP8: TestPoint, symbol Connector:TestPoint
Connections:
- new net AI_MFC_FLOW: J5.7 (Pin_7), R6.2, TP8.1
- new net AI_MFC_FLOW_FILT: C13.1, R6.1
- new net AI_PRESSURE: J5.6 (Pin_6), R5.2, TP7.1
- new net AI_PRESSURE_FILT: C12.1, R5.1
- new net AO_MFC_SETPOINT: J5.5 (Pin_5), R4.2, TP6.1
- new net AO_MFC_SP_FILT: C11.1, R4.1
- new net DO_FORELINE: J5.1 (Pin_1), R1.2, TP1.1
- new net DO_FORELINE_DRV: R1.1
- new net DO_N2: J5.3 (Pin_3), R3.2, TP4.1
- new net DO_N2_DRV: R3.1
- new net DO_PRECURSOR: J5.2 (Pin_2), R2.2, TP3.1
- new net DO_PRECURSOR_DRV: R2.1
- new net GND_SIG: C11.2, C12.2, C13.2, J5.4 (Pin_4), J5.8 (Pin_8), TP2.1, TP5.1
