File: mfc_interface.kicad_sch (KiCad schematic)
At the start: 0 parts

Commit message: complete mfc interface
Parts:
- added C11, C12: 10nF, symbol Device:C
- added C14, C16: 10µF, symbol Device:C
- added C15, C17: 0.1µF, symbol Device:C
- added J_MFC1: MFC_DB15, symbol Connector:DA15_Socket
- added R1, R2: 1kΩ, symbol Device:R
- added TP10, TP11, TP12, TP13, TP14, TP9: TestPoint, symbol Connector:TestPoint
Connections:
- new net: C12.1, J_MFC1.2, R2.2, TP9.1
- new net: C11.1, J_MFC1.8, R1.2, TP10.1
- new net: C16.2, C17.1
- new net: C14.2, C15.1
- new net +15V: C17.2, J_MFC1.7, TP12.1
- new net -15V: C15.2, J_MFC1.6, TP11.1
- new net AI_MFC_FLOW: R2.1
- new net AO_MFC_SETPOINT: R1.1
- new net CHASSIS_GND: J_MFC1.15 (P15)
- new net GND_PWR: C14.1, C16.1, J_MFC1.5
- new net GND_SIG: C11.2, C12.2, J_MFC1.11 (P111), J_MFC1.12 (P12), TP13.1, TP14.1
- no-connect marks 0 -> 7
