File: vacuum_gauge_interface.kicad_sch (KiCad schematic)
At the start: 0 parts

Commit message: add vacuum gauge interface with analog filtering and test points
Parts:
- added C18: 0.1uF, symbol Device:C
- added C19: 47uF, symbol Device:C_Polarized
- added C20: 10nF, symbol Device:C
- added J9: VACUUM_GAUGE_8PIN, symbol Connector_Generic:Conn_01x08
- added R7: 1k, symbol Device:R
- added TP15: TP_VAC_24V, symbol Connector:TestPoint
- added TP16: TP_VAC_GND, symbol Connector:TestPoint
- added TP17: TP_VAC_SIG, symbol Connector:TestPoint
- added TP18: TP_VAC_SIG_GND, symbol Connector:TestPoint
Connections:
- new net +24V: C18.1, C19.1, J9.1 (Pin_1), TP15.1
- new net AI_PRESSURE: J9.3 (Pin_3), R7.2, TP17.1
- new net AI_PRESSURE_FILT: C20.1, R7.1
- new net GND_PWR: C18.2, C19.2, J9.2 (Pin_2), TP16.1
- new net GND_SIG: C20.2, J9.4 (Pin_4), TP18.1
- no-connect marks 0 -> 4
